File: electronics/evpr.brd (EAGLE design)
At the start: 88.3 x 47 mm, 137 parts

Commit message: added manufacturing breakoffs
Routing:
- net GND: vias 164 -> 166
Other:
- board size 88.3 x 47 mm -> 88.4 x 47.3 mm
Changed lines of the file:
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@@
 <setting verticaltext="up"/>
 </settings>
-<grid distance="10" unitdist="mil" unit="mm" style="lines" multiple="1" display="yes" altdistance="1" altunitdist="mil" altunit="mil"/>
+<grid distance="10" unitdist="mil" unit="mil" style="lines" multiple="1" display="yes" altdistance="1" altunitdist="mil" altunit="mil"/>
 <layers>
 <layer number="1" name="Top" color="4" fill="1" visible="yes" active="yes"/>
@@
 <layer number="18" name="Vias" color="2" fill="1" visible="yes" active="yes"/>
 <layer number="19" name="Unrouted" color="6" fill="1" visible="no" active="yes"/>
-<layer number="20" name="Dimension" color="24" fill="1" visible="no" active="yes"/>
+<layer number="20" name="Dimension" color="24" fill="1" visible="yes" active="yes"/>
 <layer number="21" name="tPlace" color="7" fill="1" visible="yes" active="yes"/>
 <layer number="22" name="bPlace" color="7" fill="1" visible="yes" active="yes"/>
@@
 <layer number="44" name="Drills" color="7" fill="1" visible="no" active="yes"/>
 <layer number="45" name="Holes" color="7" fill="1" visible="no" active="yes"/>
-<layer number="46" name="Milling" color="3" fill="1" visible="no" active="yes"/>
+<layer number="46" name="Milling" color="3" fill="1" visible="yes" active="yes"/>
 <layer number="47" name="Measures" color="7" fill="1" visible="no" active="yes"/>
 <layer number="48" name="Document" color="7" fill="1" visible="no" active="yes"/>
@@
 <wire x1="40.005" y1="24.13" x2="40.005" y2="15.875" width="0.025" layer="52"/>
 <wire x1="19.8374" y1="-17.2212" x2="30.48" y2="-14.732" width="0.0254" layer="20" curve="140"/>
-<wire x1="19.8374" y1="-17.2212" x2="5.588" y2="-25.4" width="0.0254" layer="20"/>
 <wire x1="-5.588" y1="-28.702" x2="5.588" y2="-28.702" width="0.0254" layer="20" curve="180"/>
 <wire x1="5.588" y1="-28.702" x2="5.588" y2="-25.4" width="0.0254" layer="20"/>
@@
 <wire x1="-26.67" y1="-21.336" x2="-12.446" y2="-21.336" width="0.0254" layer="20"/>
 <wire x1="-15.494" y1="-53.848" x2="-19.558" y2="-52.832" width="0.0254" layer="20"/>
-<wire x1="-19.558" y1="-52.832" x2="-27.432" y2="-52.832" width="0.0254" layer="20"/>
-<wire x1="-27.432" y1="-52.832" x2="-27.432" y2="-44.196" width="0.0254" layer="20"/>
+<wire x1="-19.558" y1="-52.832" x2="-28.448" y2="-52.832" width="0.0254" layer="20"/>
+<wire x1="-27.432" y1="-48.006" x2="-27.432" y2="-44.196" width="0.0254" layer="20"/>
 <wire x1="-27.432" y1="-44.196" x2="-28.448" y2="-44.196" width="0.0254" layer="20"/>
 <wire x1="-1.016" y1="-56.134" x2="9.144" y2="-56.134" width="0.0254" layer="20"/>
@@
 <wire x1="30.48" y1="-14.732" x2="30.48" y2="-13.462" width="0.0254" layer="20"/>
 <wire x1="30.48" y1="-13.462" x2="44.45" y2="-13.462" width="0.0254" layer="20"/>
-<wire x1="42.672" y1="-37.338" x2="46.482" y2="-33.528" width="0.0254" layer="20"/>
 <wire x1="46.482" y1="-33.528" x2="48.006" y2="-33.528" width="0.0254" layer="20"/>
 <wire x1="47.498" y1="-10.16" x2="52.578" y2="-15.24" width="0.0254" layer="20" curve="-180"/>
@@
 </text>
 <text x="26.416" y="-43.688" size="1" layer="21" font="vector" rot="R30">EVPR 2.2.0</text>
+<wire x1="-34.798" y1="-50.546" x2="-34.798" y2="-56.388" width="0.0254" layer="20"/>
+<wire x1="-34.798" y1="-56.388" x2="-30.988" y2="-56.388" width="0.0254" layer="20"/>
+<wire x1="42.672" y1="-56.388" x2="53.594" y2="-56.388" width="0.0254" layer="20"/>
+<wire x1="53.594" y1="-56.388" x2="53.594" y2="-45.466" width="0.0254" layer="20"/>
+<wire x1="3.302" y1="-9.144" x2="-3.556" y2="-9.144" width="0.0254" layer="20"/>
+<wire x1="-34.798" y1="-50.546" x2="-32.258" y2="-48.006" width="0.0254" layer="20"/>
+<wire x1="-32.258" y1="-48.006" x2="-27.432" y2="-48.006" width="0.0254" layer="20"/>
+<wire x1="-28.448" y1="-52.832" x2="-28.448" y2="-53.848" width="0.0254" layer="20"/>
+<wire x1="-28.448" y1="-53.848" x2="-30.988" y2="-56.388" width="0.0254" layer="20"/>
+<wire x1="42.672" y1="-37.338" x2="42.672" y2="-56.388" width="0.0254" layer="20"/>
+<wire x1="53.594" y1="-45.466" x2="46.482" y2="-38.354" width="0.0254" layer="20"/>
+<wire x1="46.482" y1="-38.354" x2="46.482" y2="-33.528" width="0.0254" layer="20"/>
+<wire x1="-3.556" y1="-9.144" x2="-3.556" y2="-16.256" width="0.0254" layer="20"/>
+<wire x1="-3.556" y1="-16.256" x2="5.588" y2="-25.4" width="0.0254" layer="20"/>
+<wire x1="3.302" y1="-9.144" x2="3.302" y2="-12.7" width="0.0254" layer="20"/>
+<wire x1="3.302" y1="-12.7" x2="12.192" y2="-21.59" width="0.0254" layer="20"/>
+<wire x1="12.192" y1="-21.59" x2="19.8374" y2="-17.2212" width="0.0254" layer="20"/>
+<wire x1="6.1722" y1="-24.3586" x2="10.8204" y2="-21.717" width="0.762" layer="20"/>
+<wire x1="6.1722" y1="-24.3586" x2="10.8204" y2="-21.717" width="0.762" layer="46"/>
+<wire x1="-28.194" y1="-49.022" x2="-28.194" y2="-51.816" width="0.762" layer="20"/>
+<wire x1="-28.194" y1="-49.022" x2="-28.194" y2="-51.816" width="0.762" layer="46"/>
+<wire x1="43.688" y1="-37.592" x2="45.466" y2="-35.814" width="0.762" layer="20"/>
+<wire x1="43.688" y1="-37.592" x2="45.466" y2="-35.814" width="0.762" layer="46"/>
 </plain>
 <attributes>
@@
 <vertex x="20.486209375" y="-54.1368"/>
 </polygon>
-<wire x1="-25.908" y1="-22.352" x2="-24.7467125" y2="-14.2875" width="0" layer="19" extent="1-1"/>
+<via x="-31.816915625" y="-53.16349375" extent="1-16" drill="3.2258" diameter="4.7752"/>
+<via x="-0.066915625" y="-12.77749375" extent="1-16" drill="3.2258" diameter="4.7752"/>
+<wire x1="-26.67" y1="-45.974" x2="-31.816915625" y2="-53.16349375" width="0" layer="19" extent="1-1"/>
 <wire x1="24.7467125" y1="-14.2875" x2="21.5138" y2="-19.685" width="0" layer="19" extent="1-1"/>
 <wire x1="0" y1="-28.575" x2="-6.2738" y2="-29.1592" width="0" layer="19" extent="1-1"/>
+<wire x1="-24.7467125" y1="-14.2875" x2="-25.908" y2="-22.352" width="0" layer="19" extent="1-1"/>
+<wire x1="-0.066915625" y1="-12.77749375" x2="8.5344" y2="-24.6888" width="0" layer="19" extent="1-1"/>
 </signal>
 <signal name="VCONV">
@@
 <via x="33.4518" y="-29.845" extent="1-16" drill="0.254"/>
 </signal>
+<signal name="GND1">
+<via x="50.424928125" y="-53.1815375" extent="1-16" drill="3.2258" diameter="4.7752"/>
+</signal>
 </signals>
