File: electronics/ESP32_USB_INTERFACE_NOESP.sch (EAGLE design)
At the start: 26 parts, among them J1 10118193-0001LF, T1 MMBT2222A, T2 MMBT2222A

Commit message: Update mainboard and progboard to use smaller connector
Parts:
- XPROG: value (none) -> PR20B04HBDN; device con-lstb:MA04-2 -> mccloud:PR20B04HBDN
Changed lines of the file:
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@@
 <part name="JP1" library="jumper" library_urn="urn:adsk.eagle:library:252" deviceset="JP1E" device="" package3d_urn="urn:adsk.eagle:package:15455/1"/>
 <part name="JP2" library="jumper" library_urn="urn:adsk.eagle:library:252" deviceset="JP1E" device="" package3d_urn="urn:adsk.eagle:package:15455/1"/>
-<part name="XPROG" library="con-lstb" library_urn="urn:adsk.eagle:library:162" deviceset="MA04-2" device="" package3d_urn="urn:adsk.eagle:package:8368/1"/>
+<part name="XPROG" library="mccloud" deviceset="PR20B04HBDN" device=""/>
 <part name="R2" library="mccloud" deviceset="R0603" device="" value="10k">
 <attribute name="COMPONENT" value="RMCF0603FT10K0"/>
