File: electronics/evpr_osh.sch (EAGLE design)
At the start: 140 parts

Commit message: Update osh version
Parts:
- removed C.USB1, C.USB4: 4.7uF, mccloud:C0603
- removed C.USB2, C.USB3: 0.1uF, mccloud:C0603
- removed C.USB5: 4.7 nF, mccloud:C0603
- removed Q.ESP1: DMN5L06K-7, mccloud:DMN5L06K-7
- removed Q.USB1, Q.USB2: MMBT2222A, transistor-neu-to92:MMBT2222ALT1-NPN-SOT23-BEC
- removed R.ESP1, R.USB2, R.USB3: 10k, mccloud:R0603
- removed R.USB1: 1k, mccloud:R0603
- removed R.USB5: 22.1k, mccloud:R0603
- removed R.USB6: 47.5K, mccloud:R0603
- removed R.USB7: 1M, mccloud:R0603
- removed SJ.ESP1: (no value), jumper:SJ
- removed TP11, TP14, TP15, TP3, TP5, TP7, TP8: PTR1TP10R, testpad:PTR1TP10R
- removed U.USB1: CP2102N-A02-GQFN24R, mccloud:CP2102N-A02-GQFN24R
- removed X.ESP2: RSTBTN, mccloud:RSTBTN
- removed X.USB1: 10118193-0001LF, mccloud:10118193-0001LF
- added SV1: PR20B04HBDN, mccloud:PR20B04HBDN
Connections:
- removed net N$1: Q.ESP1.D, X.ESP2.1
- removed net N$16: R.USB1.1, U.USB1.RSTB
- removed net N$18: Q.USB1.E, R.USB3.2, TP14.TP, U.USB1.RTS
- removed net N$19: Q.USB2.E, R.USB2.2, TP8.TP, U.USB1.DTR
- removed net N$20: Q.USB1.B, R.USB2.1
- removed net N$21: Q.USB2.B, R.USB3.1
- removed net N$34: C.USB5.2, R.USB7.2, TP15.TP, X.USB1.SHIELD
- removed net N$39: R.USB1.2, U.USB1.VIO
- removed net N$40: C.USB1.2, C.USB2.2, TP3.TP, U.USB1.VDD
- removed net RST_DISABLE: Q.ESP1.G, R.ESP1.2, U.ESP1.IO18
- removed net USBD+: U.USB1.D+, X.USB1.D+
- removed net USBD-: U.USB1.D-, X.USB1.D-
- removed net USBSENSE: R.USB5.1, R.USB6.2, U.ESP1.IO20, U.USB1.VBUS
- removed net VUSB: C.USB3.2, C.USB4.2, Q.DS1.A, Q.ZZ2.A, R.USB5.2, TP7.TP, U.USB1.VREGIN, X.USB1.VUSB
- new net VPROG: Q.DS1.A, Q.ZZ2.A, SV1.6
- net BOOTMODE: now also SV1.3; no longer Q.USB2.C, TP11.TP
- net ESP_POWER: now also SV1.8; no longer R.ESP1.1
- net ESP_RX: now also SV1.5; no longer U.USB1.TXD
- net ESP_TX: now also SV1.7; no longer U.USB1.RXD
- net GND: now also SV1.2; no longer C.USB1.1, C.USB2.1, C.USB3.1, C.USB4.1, C.USB5.1, Q.ESP1.S, R.USB6.1, R.USB7.1, SJ.ESP1.1, U.USB1.GND, X.USB1.GND
- net RESET: now also SV1.1; no longer Q.USB1.C, SJ.ESP1.2, TP5.TP, X.ESP2.2
Other:
- note added: "ESP: ESP32 GPIO & Prog Interface"
- note removed: "ESP: ESP32 GPIO & Reset"
- note removed: "NOTE: LED_BUILTIN will blink during flashing. This is why the LED circuit is included here, rather than in the ESP32 block."
- note removed: "USB: USB Interface"
- moved on the sheet: D.USB1, R.ESP2, R.USB4
