File: electronics/Mini Boards (Testing)/evpr_mini.brd (EAGLE design)
At the start: 82.8 x 33.8 mm, 76 parts

Commit message: Applied changes from stencil testing. Fixed some packages. Altered functional groups. Other Misc. Changes. This is immediately before component mass renaming.
Connections:
- net N$59: now also U$3.BST; no longer U$3.TMR
- net N$7: now also U$3.TMR; no longer U$3.P$14
