File: electronics/boardfiles/evpr_mainboard.sch (EAGLE design)
At the start: 115 parts

Commit message: Add hall-effect tachometer, remove old tach, large-scale silkscreen updates, minor updates to various components, removed strange void in internal layers
Parts:
- removed C.VI1, C.VI2*: 0.1uF, mccloud:C0603
- removed R.VI4: 100k, mccloud:R0603
- removed R.VI5: 22.1k, mccloud:R0603
- removed SV1: PR20B04HBDN, mccloud:PR20B04HBDN
- removed X.ESP1: (no value), con-lsta:FE05-1
- added C.ESP5: 0.1uF, mccloud:C0603
- added R.ESP7: 100k, mccloud:R0603
- added R.ESP8*, R.ESP9*: 0, mccloud:R0603
- added U.ESP10: HALLEFFECT, mccloud:HALLEFFECT
- added X.ESP6: PR20B04HBDN, mccloud:PR20B04HBDN
- X.VI1: value B3P-VH(LF)(SN) -> 2-THROUGHOLE-OFFSET; device mccloud:B3P-VH(LF)(SN) -> mccloud:2-THROUGHOLE-OFFSET
Connections:
- removed net N$49: U.ESP1.SCS/CMD, X.ESP1.5
- removed net N$66: U.ESP1.SCL/CLK, X.ESP1.4
- removed net N$68: U.ESP1.SDO/SD0, X.ESP1.3
- removed net N$70: U.ESP1.SDI/SD1, X.ESP1.2
- removed net TACH: C.VI2*.1, R.VI4.1, R.VI5.2, U.ESP1.IO16
- removed net TACH_RAW: C.VI1.1, Q.VI1.K1, R.VI4.2, X.VI1.3
- new net HALL: R.ESP7.2, U.ESP1.IO16, U.ESP10.OUT
- new net HALL_EN: R.ESP9*.2, U.ESP1.IO14
- new net N$1: C.ESP5.2, R.ESP7.1, R.ESP8*.1, R.ESP9*.1, U.ESP10.VCC
- net BOOTMODE: now also X.ESP6.3; no longer SV1.3
- net ESP_POWER: now also R.ESP8*.2, X.ESP6.8; no longer SV1.8
- net ESP_RX: now also X.ESP6.5; no longer SV1.5
- net ESP_TX: now also X.ESP6.7; no longer SV1.7
- net GND: now also C.ESP5.1, U.ESP10.GND, X.ESP6.2; no longer C.VI1.2, C.VI2*.2, R.VI5.1, SV1.2, X.ESP1.1
- net RESET: now also X.ESP6.1; no longer SV1.1
- net VPROG: now also X.ESP6.6; no longer SV1.6
Other:
- moved on the sheet: D.USB1, R.USB4

Commit message: Update snapoffs to conform with OSH park recommendations, increase servo diameter, misc DRC corrections
Parts:
- SV2, SV3: device con-lstb:MA03-1 -> mccloud:MA03-1
Changed lines of the file:
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@@
 <part name="X.ESP6" library="mccloud" deviceset="PR20B04HBDN" device=""/>
 <part name="SUPPLY13" library="supply2" library_urn="urn:adsk.eagle:library:372" deviceset="GND" device=""/>
-<part name="SV2" library="con-lstb" library_urn="urn:adsk.eagle:library:162" deviceset="MA03-1" device="" package3d_urn="urn:adsk.eagle:package:8339/1"/>
-<part name="SV3" library="con-lstb" library_urn="urn:adsk.eagle:library:162" deviceset="MA03-1" device="" package3d_urn="urn:adsk.eagle:package:8339/1"/>
+<part name="SV2" library="mccloud" deviceset="MA03-1" device="" package3d_urn="urn:adsk.eagle:package:8339/1"/>
+<part name="SV3" library="mccloud" deviceset="MA03-1" device="" package3d_urn="urn:adsk.eagle:package:8339/1"/>
 <part name="JP1" library="pinhead" library_urn="urn:adsk.eagle:library:325" deviceset="PINHD-1X2" device="" package3d_urn="urn:adsk.eagle:package:22435/2"/>
 <part name="U.ESP10" library="mccloud" deviceset="HALLEFFECT" device=""/>

Commit message: Incrase diameter on a couple of more holes
Parts:
- JP1: device pinhead:PINHD-1X2 -> mccloud:PINHD-1X2
Changed lines of the file:
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@@
 <part name="SV2" library="mccloud" deviceset="MA03-1" device="" package3d_urn="urn:adsk.eagle:package:8339/1"/>
 <part name="SV3" library="mccloud" deviceset="MA03-1" device="" package3d_urn="urn:adsk.eagle:package:8339/1"/>
-<part name="JP1" library="pinhead" library_urn="urn:adsk.eagle:library:325" deviceset="PINHD-1X2" device="" package3d_urn="urn:adsk.eagle:package:22435/2"/>
+<part name="JP1" library="mccloud" deviceset="PINHD-1X2" device="" package3d_urn="urn:adsk.eagle:package:22435/2"/>
 <part name="U.ESP10" library="mccloud" deviceset="HALLEFFECT" device=""/>
 <part name="C.ESP5" library="mccloud" deviceset="C0603" device="" value="0.1uF">

Commit message: Various finishing touches
Parts:
- removed C.ESP5: 0.1uF, mccloud:C0603
- removed JP1: (no value), mccloud:PINHD-1X2
- removed R.ESP7: 100k, mccloud:R0603
- removed R.ESP8*, R.ESP9*: 0, mccloud:R0603
- removed U.ESP10: HALLEFFECT, mccloud:HALLEFFECT
- added C.TK1: 0.1uF, mccloud:C0603
- added R.TK1*, R.TK2: 0, mccloud:R0603
- added R.TK3: 100k, mccloud:R0603
- added SV1: (no value), mccloud:MA03-1
- added U.TK1: HALLEFFECT, mccloud:HALLEFFECT
- SV3: device mccloud:MA03-1 -> mccloud:PINHD-1X2
- renumbered R.USB4 to R.ESP1
Connections:
- net ESP_POWER: now also R.TK2.2; no longer R.ESP8*.2
- net GND: now also C.TK1.1, SV1.3, SV3.1, U.TK1.GND; no longer C.ESP5.1, JP1.1, SV3.3, U.ESP10.GND
- net HALL: now also R.TK3.2, U.TK1.OUT; no longer R.ESP7.2, U.ESP10.OUT
- net HALL_EN: now also R.TK1*.2; no longer R.ESP9*.2
- net N$1: now also C.TK1.2, R.TK1*.1, R.TK2.1, R.TK3.1, U.TK1.VCC; no longer C.ESP5.2, R.ESP7.1, R.ESP8*.1, R.ESP9*.1, U.ESP10.VCC
- net N$12: now also SV1.1; no longer SV3.1
- net SYS_POWER: now also SV1.2; no longer JP1.2
Other:
- note added: "TK: Tachometer"
