File: electronics/boardfiles/evpr_programmer.brd (EAGLE design)
At the start: 44.2 x 25.4 mm, 26 parts, among them J1 10118193-0001LF, T1 MMBT2222A, T2 MMBT2222A

Commit message: Various finishing touches
Parts:
- renumbered U$1 to U1
Changed lines of the file:
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@@
 <attribute name="VALUE" x="27.305" y="40.64" size="0.8128" layer="27" font="vector" ratio="15"/>
 </element>
-<element name="U$1" library="mccloud" package="QFN24-4X4" value="CP2102N-A02-GQFN24R" x="34.036" y="44.196" smashed="yes" rot="R270">
+<element name="U1" library="mccloud" package="QFN24-4X4" value="CP2102N-A02-GQFN24R" x="34.036" y="44.196" smashed="yes" rot="R270">
 <attribute name="NAME" x="33.814" y="40.6" size="0.8128" layer="25" font="vector" ratio="15"/>
 <attribute name="VALUE" x="30.286" y="46.196" size="0.8128" layer="27" font="vector" ratio="15" rot="R270"/>
 </element>
 <element name="RESET" library="mccloud" package="PTS645" value="MOMENTARY_SWITCH" x="44.196" y="37.084" smashed="yes" rot="R180">
+<attribute name="COMPONENT" value="PTS645" x="44.196" y="37.084" size="1.778" layer="27" rot="R180" display="off"/>
 <attribute name="NAME" x="46.99" y="33.909" size="0.8128" layer="25" font="vector" ratio="15" rot="R180"/>
 </element>
@@
 <signal name="N$3">
 <contactref element="R1" pad="1"/>
-<contactref element="U$1" pad="9"/>
+<contactref element="U1" pad="9"/>
 <contactref element="TP1" pad="TP"/>
 <wire x1="26.504" y1="46.736" x2="26.8314" y2="47.0634" width="0.254" layer="1"/>
@@
 </signal>
 <signal name="RX">
-<contactref element="U$1" pad="20"/>
+<contactref element="U1" pad="20"/>
 <contactref element="XPROG" pad="P$7"/>
 <contactref element="XDEBG" pad="8"/>
@@
 </signal>
 <signal name="TX">
-<contactref element="U$1" pad="21"/>
+<contactref element="U1" pad="21"/>
 <contactref element="XPROG" pad="P$5"/>
 <contactref element="XDEBG" pad="6"/>
@@
 </signal>
 <signal name="RTS">
-<contactref element="U$1" pad="23"/>
+<contactref element="U1" pad="23"/>
 <contactref element="R2" pad="1"/>
 <contactref element="T2" pad="E"/>
@@
 </signal>
 <signal name="DTR">
-<contactref element="U$1" pad="19"/>
+<contactref element="U1" pad="19"/>
 <contactref element="T1" pad="E"/>
 <contactref element="R3" pad="1"/>
@@
 <contactref element="J1" pad="5"/>
 <contactref element="R6" pad="2"/>
-<contactref element="U$1" pad="2"/>
-<contactref element="U$1" pad="EXP"/>
+<contactref element="U1" pad="2"/>
+<contactref element="U1" pad="EXP"/>
 <contactref element="C2" pad="1"/>
 <contactref element="C3" pad="2"/>
@@
 </signal>
 <signal name="N$11">
-<contactref element="U$1" pad="3"/>
+<contactref element="U1" pad="3"/>
 <contactref element="J1" pad="3"/>
 <contactref element="TP2" pad="TP"/>
@@
 </signal>
 <signal name="N$12">
-<contactref element="U$1" pad="4"/>
+<contactref element="U1" pad="4"/>
 <contactref element="J1" pad="2"/>
 <contactref element="TP3" pad="TP"/>
@@
 <signal name="N$14">
 <contactref element="R6" pad="1"/>
-<contactref element="U$1" pad="8"/>
+<contactref element="U1" pad="8"/>
 <contactref element="R5" pad="2"/>
 <contactref element="TP4" pad="TP"/>
@@
 </signal>
 <signal name="N$13">
-<contactref element="U$1" pad="7"/>
+<contactref element="U1" pad="7"/>
 <contactref element="JP3" pad="2"/>
 <wire x1="24.892" y1="37.846" x2="26.67" y2="39.624" width="0.254" layer="1"/>
@@
 </signal>
 <signal name="N$2">
-<contactref element="U$1" pad="6"/>
+<contactref element="U1" pad="6"/>
 <contactref element="JP2" pad="2"/>
 <wire x1="32.786" y1="46.146" x2="32.786" y2="46.4" width="0.254" layer="1"/>
@@
 <signal name="N$4">
 <contactref element="JP1" pad="2"/>
-<contactref element="U$1" pad="5"/>
+<contactref element="U1" pad="5"/>
 <contactref element="R1" pad="2"/>
 <wire x1="24.804" y1="46.736" x2="24.892" y2="46.648" width="0.254" layer="1"/>
